Commit message: Add autonomy navigation stack, mission-control dashboards, and field robot model
Introduce nav mission executor and pure helpers, navigation controller with local
terrain corridor planning, global mapper TF and occupancy codec paths, and dig
sequence gating on the local terrain grid. Extend autonomy supervisor and shadow
logic, mission bridge snapshot contract, and offline tests.

Mission-control gains Nav and Dig sequence charts, dig/dump mission chart, demo
mode wiring, and bridge contract updates. Lunar CLI adds run session logging and
nav-dig launch flags; Makefile documents LUNAR_RUN_FLAGS and log packaging.

URDF: field footprint (0.68 m × 1.44 m), base_footprint under geometric centroid,
Nav2 and global_costmapper clearance from robot_footprint. Default global map
extent matches a 10.5 m arena span. Ignore stray root uv.lock.

Co-authored-by: Cursor <cursoragent@cursor.com>

File: src/backend/description/robot.urdf.xacro (robot description, xacro)
@@ -13,4 +13,6 @@
     <xacro:include filename="robot_wheel.xacro" />
     <xacro:include filename="robot_inertia.xacro" />
+    <!-- base_link origin: horizontal centroid of plan-view chassis box; z = box center (URDF box centered on link). -->
+    <!-- base_link origin: centroid of the plan-view chassis box (XY) and of that box in Z. -->
     <link name="base_link">
         <!-- Base -->
@@ -50,4 +52,11 @@
         <xacro:inertial_box mass="${base_mass}" x="${base_length}" y="${base_width}" z="${base_height}"/>
     </link>
+    <!-- Horizontal projection of base_link centroid onto the ground (same X,Y as base_link). -->
+    <link name="base_footprint"/>
+    <joint name="base_footprint_joint" type="fixed">
+        <parent link="base_link"/>
+        <child link="base_footprint"/>
+        <origin xyz="0 0 ${-base_link_to_ground_m}" rpy="0 0 0"/>
+    </joint>
     <xacro:include filename="robot_actuator.xacro"   />
     <!-- xacro:include filename="robot_imu.xacro"       / -->

File: src/backend/description/robot_properties.xacro (robot description, xacro)
@@ -5,6 +5,9 @@
     <xacro:property name="wheel_height"    value="0.062"/>
     <xacro:property name="wheel_mass"      value="100.83"/>
-    <xacro:property name="base_width"      value="0.483"/>
-    <xacro:property name="base_length"     value="0.711"/>
+    <!-- Ground plane under base_link origin: wheel joint z=-wheel_height, axle ~horizontal, contact ≈ -wheel_height - wheel_radius -->
+    <xacro:property name="base_link_to_ground_m" value="${wheel_height + wheel_radius}"/>
+    <!-- base_link box: X = forward/back, Y = lateral (field: 68 cm × 144 cm) -->
+    <xacro:property name="base_width"      value="1.44"/>
+    <xacro:property name="base_length"     value="0.68"/>
     <xacro:property name="base_height"     value="0.124"/>
     <xacro:property name="base_mass"       value="56.7"/>
@@ -15,3 +18,5 @@
     <xacro:property name="imu_y"           value="0.0"/>
     <xacro:property name="imu_z"           value="0.0"/>
+    <!-- Ground point under base_link centroid (wheel joint z = -wheel_height, axle ~horizontal). -->
+    <xacro:property name="base_link_to_ground_m" value="${wheel_height + wheel_radius}"/>
 </robot>

File: src/backend/description/sim_robot.urdf.xacro (robot description, xacro)
@@ -14,4 +14,5 @@
     <xacro:include filename="robot_inertia.xacro" />
     <xacro:include filename="robot_servo.xacro" />
+    <!-- base_link origin: centroid of the plan-view chassis box (XY) and of that box in Z. -->
     <link name="base_link">
         <!-- Base -->
@@ -51,4 +52,10 @@
         <xacro:inertial_box mass="${base_mass}" x="${base_length}" y="${base_width}" z="${base_height}"/>
     </link>
+    <link name="base_footprint"/>
+    <joint name="base_footprint_joint" type="fixed">
+        <parent link="base_link"/>
+        <child link="base_footprint"/>
+        <origin xyz="0 0 ${-base_link_to_ground_m}" rpy="0 0 0"/>
+    </joint>
     <!-- xacro:include filename="robot_imu.xacro"       / -->
     <xacro:include filename="robot_depth.xacro"     />
